Commit message: Right finger able to feel collisions

File: franka_description/robots/panda.gazebo.xacro (robot description, xacro)
@@ -2,4 +2,24 @@
 <robot xmlns:xacro="http://www.ros.org/wiki/xacro">
     <xacro:macro name="panda_gazebo" params="robot_name">
+		<gazebo reference="panda_rightfinger">
+			<sensor type="contact" name="main_bumper">
+				<topic>/bump_topic/rf</topic>
+				<plugin name="gazebo_ros_bumper_controller_rf" filename="libgazebo_ros_bumper.so">
+					<topic>/bump_topic/rf</topic>
+					<alwaysOn>1</alwaysOn>
+					<updateRate>100.0</updateRate>
+					<bumperTopicName>/panda/bumper/rf</bumperTopicName>
+<!--
+					<frameName>ttest</frameName>
+-->
+				</plugin>
+				<contact>
+					<collision>panda_rightfinger_collision</collision>
+					<topic>/bump_topic/rf</topic>
+				</contact>
+				<alwaysOn>true</alwaysOn>
+				<updateRate>10.0</updateRate>
+			</sensor>
+		</gazebo>
         <!-- Link0 -->
         <gazebo reference="${robot_name}_link0">

Commit message: Added xacro to make sensing available on all links

File: franka_description/robots/panda.gazebo.xacro (robot description, xacro)
@@ -2,24 +2,34 @@
 <robot xmlns:xacro="http://www.ros.org/wiki/xacro">
     <xacro:macro name="panda_gazebo" params="robot_name">
-		<gazebo reference="panda_rightfinger">
-			<sensor type="contact" name="main_bumper">
-				<topic>/bump_topic/rf</topic>
-				<plugin name="gazebo_ros_bumper_controller_rf" filename="libgazebo_ros_bumper.so">
-					<topic>/bump_topic/rf</topic>
-					<alwaysOn>1</alwaysOn>
-					<updateRate>100.0</updateRate>
-					<bumperTopicName>/panda/bumper/rf</bumperTopicName>
-<!--
-					<frameName>ttest</frameName>
--->
-				</plugin>
-				<contact>
-					<collision>panda_rightfinger_collision</collision>
-					<topic>/bump_topic/rf</topic>
-				</contact>
-				<alwaysOn>true</alwaysOn>
-				<updateRate>10.0</updateRate>
-			</sensor>
-		</gazebo>
+		<xacro:macro name="add_collision_sensing" params="link_name">
+			<gazebo reference="${link_name}">
+				<sensor type="contact" name="${link_name}_bumper">
+					<topic>/bump_topic/${link_name}</topic>
+					<plugin name="gazebo_ros_bumper_controller_${link_name}" filename="libgazebo_ros_bumper.so">
+						<topic>/bump_topic/${link_name}</topic>
+						<alwaysOn>1</alwaysOn>
+						<updateRate>100.0</updateRate>
+						<bumperTopicName>/panda/bumper/${link_name}</bumperTopicName>
+					</plugin>
+					<contact>
+						<collision>${link_name}_collision</collision>
+						<topic>/bump_topic/${link_name}</topic>
+					</contact>
+					<alwaysOn>true</alwaysOn>
+					<updateRate>10.0</updateRate>
+				</sensor>
+			</gazebo>
+		</xacro:macro>
+		<xacro:add_collision_sensing link_name="${robot_name}_link1"/>
+		<xacro:add_collision_sensing link_name="${robot_name}_link2"/>
+		<xacro:add_collision_sensing link_name="${robot_name}_link3"/>
+		<xacro:add_collision_sensing link_name="${robot_name}_link4"/>
+		<xacro:add_collision_sensing link_name="${robot_name}_link5"/>
+		<xacro:add_collision_sensing link_name="${robot_name}_link6"/>
+		<xacro:add_collision_sensing link_name="${robot_name}_link7"/>
+		<xacro:add_collision_sensing link_name="${robot_name}_link8"/>
+		<xacro:add_collision_sensing link_name="${robot_name}_hand"/>
+		<xacro:add_collision_sensing link_name="${robot_name}_rightfinger"/>
+		<xacro:add_collision_sensing link_name="${robot_name}_leftfinger"/>
         <!-- Link0 -->
         <gazebo reference="${robot_name}_link0">

Commit message: Added second part of link 7 collision mesh

File: franka_description/robots/panda.gazebo.xacro (robot description, xacro)
@@ -14,4 +14,7 @@
 					<contact>
 						<collision>${link_name}_collision</collision>
+						<xacro:if value="${'panda_link7'==link_name}">
+							<collision>panda_link7_fixed_joint_lump__panda_hand_collision_1</collision>
+						</xacro:if>
 						<topic>/bump_topic/${link_name}</topic>
 					</contact>
