Commit message: Added a probing tool to frankas hand

File: franka_description/robots/hand.xacro (robot description, xacro)
@@ -82,4 +82,50 @@
       <limit effort="20" lower="0.0" upper="0.04" velocity="0.2"/>
     </joint>
+    <joint name="${ns}_probe_cyl_joint" type="fixed">
+      <parent link="${ns}_hand"/>
+      <child link="${ns}_probe_cyl"/>
+      <origin xyz="0 0 0.12" rpy="0 0 0"/>
+      <axis xyz="0 1 0"/>
+    </joint>
+    <link name="${ns}_probe_cyl">
+	  <visual>
+	    <geometry>
+		  <cylinder length="0.1" radius="0.01"/>
+	    </geometry>
+	  </visual>
+      <collision>
+		<geometry>
+	      <cylinder length="0.1" radius="0.01"/>
+	    </geometry>
+      </collision>
+      <inertial>
+        <origin xyz="0 0 0" rpy="0 0 0" />
+        <mass value="0.01" />
+        <inertia ixx="0.1" ixy="0.0" ixz="0.0" iyy="0.1" iyz="0.0" izz="0.1" />
+      </inertial>
+    </link>
+    <joint name="${ns}_probe_ball_joint" type="fixed">
+      <parent link="${ns}_probe_cyl"/>
+      <child link="${ns}_probe_ball"/>
+      <origin xyz="0 0 0.07" rpy="0 0 0"/>
+      <axis xyz="0 1 0"/>
+    </joint>
+    <link name="${ns}_probe_ball">
+      <visual>
+        <geometry>
+		  <sphere radius="0.03"/>
+        </geometry>
+      </visual>
+      <collision>
+		<geometry>
+	      <sphere radius="0.03"/>
+	    </geometry>
+      </collision>
+      <inertial>
+        <origin xyz="0 0 0" rpy="0 0 0" />
+        <mass value="0.01" />
+        <inertia ixx="0.1" ixy="0.0" ixz="0.0" iyy="0.1" iyz="0.0" izz="0.1" />
+      </inertial>
+    </link>
   </xacro:macro>
 </robot>

File: franka_description/robots/panda.gazebo.xacro (robot description, xacro)
@@ -16,4 +16,10 @@
 						<xacro:if value="${'panda_link7'==link_name}">
 							<collision>panda_link7_fixed_joint_lump__panda_hand_collision_1</collision>
+						</xacro:if>
+						<xacro:if value="${'panda_probe_cyl'==link_name}">
+							<collision>panda_link7_fixed_joint_lump__panda_probe_cyl_collision_2</collision>
+						</xacro:if>
+						<xacro:if value="${'panda_probe_ball'==link_name}">
+							<collision>panda_link7_fixed_joint_lump__panda_probe_ball_collision_3</collision>
 						</xacro:if>
 						<topic>/bump_topic/${link_name}</topic>
@@ -35,4 +41,6 @@
 		<xacro:add_collision_sensing link_name="${robot_name}_rightfinger"/>
 		<xacro:add_collision_sensing link_name="${robot_name}_leftfinger"/>
+		<xacro:add_collision_sensing link_name="${robot_name}_probe_cyl"/>
+		<xacro:add_collision_sensing link_name="${robot_name}_probe_ball"/>
         <!-- Link0 -->
         <gazebo reference="${robot_name}_link0">

Commit message: Added force torque sensing for probe

File: franka_description/robots/hand.xacro (robot description, xacro)
@@ -82,9 +82,10 @@
       <limit effort="20" lower="0.0" upper="0.04" velocity="0.2"/>
     </joint>
-    <joint name="${ns}_probe_cyl_joint" type="fixed">
+    <joint name="${ns}_probe_cyl_joint" type="revolute">
       <parent link="${ns}_hand"/>
       <child link="${ns}_probe_cyl"/>
       <origin xyz="0 0 0.12" rpy="0 0 0"/>
       <axis xyz="0 1 0"/>
+      <limit effort="20" lower="0.0" upper="0.0" velocity="0.0"/>
     </joint>
     <link name="${ns}_probe_cyl">

File: franka_description/robots/panda.gazebo.xacro (robot description, xacro)
@@ -18,8 +18,8 @@
 						</xacro:if>
 						<xacro:if value="${'panda_probe_cyl'==link_name}">
-							<collision>panda_link7_fixed_joint_lump__panda_probe_cyl_collision_2</collision>
+							<collision>panda_probe_cyl_collision</collision>
 						</xacro:if>
 						<xacro:if value="${'panda_probe_ball'==link_name}">
-							<collision>panda_link7_fixed_joint_lump__panda_probe_ball_collision_3</collision>
+							<collision>panda_probe_cyl_fixed_joint_lump__panda_probe_ball_collision_1</collision>
 						</xacro:if>
 						<topic>/bump_topic/${link_name}</topic>
@@ -43,4 +43,14 @@
 		<xacro:add_collision_sensing link_name="${robot_name}_probe_cyl"/>
 		<xacro:add_collision_sensing link_name="${robot_name}_probe_ball"/>
+		<gazebo reference="${robot_name}_probe_cyl_joint">
+			<provideFeedback>true</provideFeedback>
+		</gazebo>
+		<gazebo>
+			<plugin name="ft_sensor_tool" filename="libgazebo_ros_ft_sensor.so">
+				<updateRate>100.0</updateRate>
+				<topicName>${robot_name}/ft/tool</topicName>
+				<jointName>${robot_name}_probe_cyl_joint</jointName>
+			</plugin>
+		</gazebo>
         <!-- Link0 -->
         <gazebo reference="${robot_name}_link0">

File: franka_description/robots/panda.transmission.xacro (robot description, xacro)
@@ -99,4 +99,14 @@
                 </actuator>
             </transmission>
+            <transmission name="${robot_name}_probe">
+                <type>transmission_interface/SimpleTransmission</type>
+                <joint name="${robot_name}_probe_cyl_joint">
+                    <hardwareInterface>hardware_interface/EffortJointInterface</hardwareInterface>
+                </joint>
+                <actuator name="${robot_name}_probe_cyl_joint">
+                    <hardwareInterface>hardware_interface/EffortJointInterface</hardwareInterface>
+                    <mechanicalReduction>1</mechanicalReduction>
+                </actuator>
+            </transmission>
         </xacro:if>
     </xacro:macro>

Commit message: Adapted inertias and sensor to more realistic values

File: franka_description/robots/hand.xacro (robot description, xacro)
@@ -89,4 +89,14 @@
       <limit effort="20" lower="0.0" upper="0.0" velocity="0.0"/>
     </joint>
+    <!--
+    Masses and inertia based on density of PLA (1250 kg/m^3)
+    Assumed uniform density
+    R = 0.03 m of ball
+    r = 0.01 m of cyl
+    L = 0.1 m of cyl
+    I_ball = 2./5.*m_ball*R**2
+    I_axis = 1./2.*m_cyl*r**2
+    I_oAxis = 1./4.*m_cyl*r**2+1./12.*m_cyl*L**2
+    -->
     <link name="${ns}_probe_cyl">
 	  <visual>
@@ -102,6 +112,6 @@
       <inertial>
         <origin xyz="0 0 0" rpy="0 0 0" />
-        <mass value="0.01" />
-        <inertia ixx="0.1" ixy="0.0" ixz="0.0" iyy="0.1" iyz="0.0" izz="0.1" />
+        <mass value="0.03926990816987242" />
+        <inertia ixx="3.3706671179140497e-05" ixy="0.0" ixz="0.0" iyy="3.3706671179140497e-05" iyz="0.0" izz="1.963495408493621e-06" />
       </inertial>
     </link>
@@ -125,6 +135,6 @@
       <inertial>
         <origin xyz="0 0 0" rpy="0 0 0" />
-        <mass value="0.01" />
-        <inertia ixx="0.1" ixy="0.0" ixz="0.0" iyy="0.1" iyz="0.0" izz="0.1" />
+        <mass value="0.033749999999999995" />
+        <inertia ixx="1.2149999999999997e-05" ixy="0.0" ixz="0.0" iyy="1.2149999999999997e-05" iyz="0.0" izz="1.2149999999999997e-05" />
       </inertial>
     </link>

File: franka_description/robots/panda.gazebo.xacro (robot description, xacro)
@@ -48,5 +48,5 @@
 		<gazebo>
 			<plugin name="ft_sensor_tool" filename="libgazebo_ros_ft_sensor.so">
-				<updateRate>100.0</updateRate>
+				<updateRate>1000.0</updateRate>
 				<topicName>${robot_name}/ft/tool</topicName>
 				<jointName>${robot_name}_probe_cyl_joint</jointName>

Commit message: Added a camera to the robot hand

File: franka_description/robots/hand.xacro (robot description, xacro)
@@ -82,4 +82,28 @@
       <limit effort="20" lower="0.0" upper="0.04" velocity="0.2"/>
     </joint>
+    <!-- Wrist mounted camera -->
+    <joint name="${ns}_camera_joint" type="fixed">
+      <parent link="${ns}_hand"/>
+      <child link="${ns}_camera"/>
+      <origin xyz="0.05 0 0.05" rpy="3.141 -1.57 0"/>
+      <axis xyz="0 1 0"/>
+    </joint>
+    <link name="${ns}_camera">
+	  <visual>
+	    <geometry>
+		  <box size="0.05 0.05 0.05"/>
+	    </geometry>
+	  </visual>
+      <collision>
+		<geometry>
+	      <box size="0.05 0.05 0.05"/>
+	    </geometry>
+      </collision>
+      <inertial>
+        <origin xyz="0 0 0" rpy="0 0 0" />
+        <mass value="0.15625" />
+        <inertia ixx="0.000065104" ixy="0.0" ixz="0.0" iyy="0.000065104" iyz="0.0" izz="0.000065104" />
+      </inertial>
+    </link>
     <joint name="${ns}_probe_cyl_joint" type="revolute">
       <parent link="${ns}_hand"/>

File: franka_description/robots/panda.gazebo.xacro (robot description, xacro)
@@ -2,4 +2,5 @@
 <robot xmlns:xacro="http://www.ros.org/wiki/xacro">
     <xacro:macro name="panda_gazebo" params="robot_name">
+		<!-- Add bumpers to whole robot -->
 		<xacro:macro name="add_collision_sensing" params="link_name">
 			<gazebo reference="${link_name}">
@@ -23,4 +24,7 @@
 							<collision>panda_probe_cyl_fixed_joint_lump__panda_probe_ball_collision_1</collision>
 						</xacro:if>
+						<xacro:if value="${'panda_camera'==link_name}">
+							<collision>panda_link7_fixed_joint_lump__panda_camera_collision_2</collision>
+						</xacro:if>
 						<topic>/bump_topic/${link_name}</topic>
 					</contact>
@@ -43,4 +47,6 @@
 		<xacro:add_collision_sensing link_name="${robot_name}_probe_cyl"/>
 		<xacro:add_collision_sensing link_name="${robot_name}_probe_ball"/>
+		<xacro:add_collision_sensing link_name="${robot_name}_camera"/>
+		<!-- FT sensing at probe -->
 		<gazebo reference="${robot_name}_probe_cyl_joint">
 			<provideFeedback>true</provideFeedback>
@@ -52,4 +58,53 @@
 				<jointName>${robot_name}_probe_cyl_joint</jointName>
 			</plugin>
+		</gazebo>
+		<!-- Camera -->
+		<gazebo reference="${robot_name}_camera">
+			<material>Gazebo/Red</material>
+			<sensor type="depth" name="depth_camera">
+				<always_on>true</always_on>
+				<visualize>true</visualize>
+				<update_rate>30.0</update_rate>
+				<topic>${robot_name}/depth_camera/depth_image</topic>
+				<camera name="head_depth">
+					<horizontal_fov>1.047198</horizontal_fov>
+					<image>
+						<width>640</width>
+						<height>480</height>
+						<format>R8G8B8</format>
+					</image>
+					<depth_camera></depth_camera>
+					<clip>
+						<near>0.05</near>
+						<far>3</far>
+					</clip>
+				</camera>
+				<plugin name="camera_plugin" filename="libgazebo_ros_openni_kinect.so">
+					<baseline>0.2</baseline>
+					<alwaysOn>true</alwaysOn>
+					<!-- Keep this zero, update_rate in the parent <sensor> tag
+					will control the frame rate. -->
+					<updateRate>0.0</updateRate>
+					<robotNamespace>${robot_name}</robotNamespace>
+					<cameraName>depth_camera</cameraName>
+					<imageTopicName>image</imageTopicName>
+					<cameraInfoTopicName>camera_info</cameraInfoTopicName>
+					<depthImageTopicName>depth_image</depthImageTopicName>
+					<depthImageInfoTopicName>depth_camera_info</depthImageInfoTopicName>
+					<pointCloudTopicName>points</pointCloudTopicName>
+					<frameName>${robot_name}_camera</frameName>
+					<pointCloudCutoff>0.05</pointCloudCutoff>
+					<distortionK1>0</distortionK1>
+					<distortionK2>0</distortionK2>
+					<distortionK3>0</distortionK3>
+					<distortionT1>0</distortionT1>
+					<distortionT2>0</distortionT2>
+					<CxPrime>0</CxPrime>
+					<Cx>0</Cx>
+					<Cy>0</Cy>
+					<focalLength>0</focalLength>
+					<hackBaseline>0</hackBaseline>
+				</plugin>
+			</sensor>
 		</gazebo>
         <!-- Link0 -->

Commit message: Refined inertias

File: franka_description/robots/hand.xacro (robot description, xacro)
@@ -24,5 +24,5 @@
         <origin xyz="0 0 0" rpy="0 0 0" />
         <mass value="0.68" />
-        <inertia ixx="0.1" ixy="0.0" ixz="0.0" iyy="0.1" iyz="0.0" izz="0.1" />
+        <inertia ixx="0.0013307028" ixy="0.0" ixz="0.0" iyy="0.0013307028" iyz="0.0" izz="0.0013307028" />
       </inertial>
       <!-- end for simulation -->
@@ -43,5 +43,5 @@
         <origin xyz="0 0 0" rpy="0 0 0" />
         <mass value="0.01" />
-        <inertia ixx="0.1" ixy="0.0" ixz="0.0" iyy="0.1" iyz="0.0" izz="0.1" />
+        <inertia ixx="1.6848e-06" ixy="0.0" ixz="0.0" iyy="1.6848e-06" iyz="0.0" izz="1.6848e-06" />
       </inertial>
       <!-- end for simulation -->
@@ -64,5 +64,5 @@
         <origin xyz="0 0 0" rpy="0 0 0" />
         <mass value="0.01" />
-        <inertia ixx="0.1" ixy="0.0" ixz="0.0" iyy="0.1" iyz="0.0" izz="0.1" />
+        <inertia ixx="1.6848e-06" ixy="0.0" ixz="0.0" iyy="1.6848e-06" iyz="0.0" izz="1.6848e-06" />
       </inertial>
       <!-- end for simulation -->

File: franka_description/robots/panda.transmission.xacro (robot description, xacro)
@@ -7,4 +7,7 @@
                 <!-- <robotNamespace>/${robot_name}</robotNamespace> -->
             </plugin>
+            <plugin name="gravity_compensation" filename="libGravityCompensationPlugin.so">
+				<uri>model://panda</uri>
+			</plugin>
         </gazebo>
         <transmission name="${robot_name}_tran_1">

File: franka_description/robots/panda_arm.xacro (robot description, xacro)
@@ -33,5 +33,5 @@
         <origin xyz="0 0 0" rpy="0 0 0" />
         <mass value="3.06" />
-        <inertia ixx="0.3" ixy="0.0" ixz="0.0" iyy="0.3" iyz="0.0" izz="0.3" />
+        <inertia ixx="0.0060045972" ixy="0.0" ixz="0.0" iyy="0.0060045972" iyz="0.0" izz="0.0060045972" />
       </inertial>
       <!-- end for simulation -->
@@ -52,5 +52,5 @@
         <origin xyz="0 0 0" rpy="0 0 0" />
         <mass value="2.34" />
-        <inertia ixx="0.3" ixy="0.0" ixz="0.0" iyy="0.3" iyz="0.0" izz="0.3" />
+        <inertia ixx="0.0045956316" ixy="0.0" ixz="0.0" iyy="0.0045956316" iyz="0.0" izz="0.0045956316" />
       </inertial>
       <!-- end for simulation -->
@@ -82,5 +82,5 @@
         <origin xyz="0 0 0" rpy="0 0 0" />
         <mass value="2.36" />
-        <inertia ixx="0.3" ixy="0.0" ixz="0.0" iyy="0.3" iyz="0.0" izz="0.3" />
+        <inertia ixx="0.0046337144" ixy="0.0" ixz="0.0" iyy="0.0046337144" iyz="0.0" izz="0.0046337144" />
       </inertial>
       <!-- end for simulation -->
@@ -112,5 +112,5 @@
         <origin xyz="0 0 0" rpy="0 0 0" />
         <mass value="2.38" />
-        <inertia ixx="0.3" ixy="0.0" ixz="0.0" iyy="0.3" iyz="0.0" izz="0.3" />
+        <inertia ixx="0.00466578" ixy="0.0" ixz="0.0" iyy="0.00466578" iyz="0.0" izz="0.00466578" />
       </inertial>
       <!-- end for simulation -->
@@ -142,5 +142,5 @@
         <origin xyz="0 0 0" rpy="0 0 0" />
         <mass value="2.43" />
-        <inertia ixx="0.3" ixy="0.0" ixz="0.0" iyy="0.3" iyz="0.0" izz="0.3" />
+        <inertia ixx="0.0047579784" ixy="0.0" ixz="0.0" iyy="0.0047579784" iyz="0.0" izz="0.0047579784" />
       </inertial>
       <!-- end for simulation -->
@@ -172,5 +172,5 @@
         <origin xyz="0 0 0" rpy="0 0 0" />
         <mass value="3.5" />
-        <inertia ixx="0.3" ixy="0.0" ixz="0.0" iyy="0.3" iyz="0.0" izz="0.3" />
+        <inertia ixx="0.0068523756" ixy="0.0" ixz="0.0" iyy="0.0068523756" iyz="0.0" izz="0.0068523756" />
       </inertial>
       <!-- end for simulation -->
@@ -202,5 +202,5 @@
         <origin xyz="0 0 0" rpy="0 0 0" />
         <mass value="1.47" />
-        <inertia ixx="0.3" ixy="0.0" ixz="0.0" iyy="0.3" iyz="0.0" izz="0.3" />
+        <inertia ixx="0.0028760256" ixy="0.0" ixz="0.0" iyy="0.0028760256" iyz="0.0" izz="0.0028760256" />
       </inertial>
       <!-- end for simulation -->
@@ -232,5 +232,5 @@
         <origin xyz="0 0 0" rpy="0 0 0" />
         <mass value="0.45" />
-        <inertia ixx="0.3" ixy="0.0" ixz="0.0" iyy="0.3" iyz="0.0" izz="0.3" />
+        <inertia ixx="0.0008938776" ixy="0.0" ixz="0.0" iyy="0.0008938776" iyz="0.0" izz="0.0008938776" />
       </inertial>
       <!-- end for simulation -->
@@ -252,5 +252,5 @@
         <origin xyz="0 0 0" rpy="0 0 0" />
         <mass value="0.0" />
-        <inertia ixx="0.3" ixy="0.0" ixz="0.0" iyy="0.3" iyz="0.0" izz="0.3" />
+        <inertia ixx="0.0" ixy="0.0" ixz="0.0" iyy="0.0" iyz="0.0" izz="0.0" />
       </inertial>
       <!-- end for simulation -->

Commit message: Enlarge camera to represent real one

File: franka_description/robots/hand.xacro (robot description, xacro)
@@ -92,10 +92,10 @@
 	  <visual>
 	    <geometry>
-		  <box size="0.05 0.05 0.05"/>
+		  <box size="0.05 0.10 0.075"/> <!-- D435 dimensions: 90 mm x 25 mm x 25 mm ; Standoff 5 cm -->
 	    </geometry>
 	  </visual>
       <collision>
 		<geometry>
-	      <box size="0.05 0.05 0.05"/>
+	      <box size="0.05 0.10 0.075"/>
 	    </geometry>
       </collision>
