Commit message: a bit less vibrations with more damping

File: franka_description/robots/panda_arm.xacro (robot description, xacro)
@@ -16,5 +16,5 @@
       <origin xyz="0.0 0.0 0.0" rpy="0.0 0.0 0.0" />
     </joint>
-    <xacro:property name="joint_damping" value="1.0"/>
+    <xacro:property name="joint_damping" value="2.0"/>
     <!-- end for simulation -->
     <link name="${arm_id}_link0">

Commit message: Rolled back inertia changes, were uncontrollable

File: franka_description/robots/panda_arm.xacro (robot description, xacro)
@@ -33,5 +33,8 @@
         <origin xyz="0 0 0" rpy="0 0 0" />
         <mass value="3.06" />
+<!--
         <inertia ixx="0.0060045972" ixy="0.0" ixz="0.0" iyy="0.0060045972" iyz="0.0" izz="0.0060045972" />
+-->
+		<inertia ixx="0.3" ixy="0.0" ixz="0.0" iyy="0.3" iyz="0.0" izz="0.3" />
       </inertial>
       <!-- end for simulation -->
@@ -52,5 +55,8 @@
         <origin xyz="0 0 0" rpy="0 0 0" />
         <mass value="2.34" />
+<!--
         <inertia ixx="0.0045956316" ixy="0.0" ixz="0.0" iyy="0.0045956316" iyz="0.0" izz="0.0045956316" />
+-->
+		<inertia ixx="0.3" ixy="0.0" ixz="0.0" iyy="0.3" iyz="0.0" izz="0.3" />
       </inertial>
       <!-- end for simulation -->
@@ -82,5 +88,8 @@
         <origin xyz="0 0 0" rpy="0 0 0" />
         <mass value="2.36" />
+<!--
         <inertia ixx="0.0046337144" ixy="0.0" ixz="0.0" iyy="0.0046337144" iyz="0.0" izz="0.0046337144" />
+-->
+		<inertia ixx="0.3" ixy="0.0" ixz="0.0" iyy="0.3" iyz="0.0" izz="0.3" />
       </inertial>
       <!-- end for simulation -->
@@ -112,5 +121,8 @@
         <origin xyz="0 0 0" rpy="0 0 0" />
         <mass value="2.38" />
+<!--
         <inertia ixx="0.00466578" ixy="0.0" ixz="0.0" iyy="0.00466578" iyz="0.0" izz="0.00466578" />
+-->
+		<inertia ixx="0.3" ixy="0.0" ixz="0.0" iyy="0.3" iyz="0.0" izz="0.3" />
       </inertial>
       <!-- end for simulation -->
@@ -142,5 +154,8 @@
         <origin xyz="0 0 0" rpy="0 0 0" />
         <mass value="2.43" />
+<!--
         <inertia ixx="0.0047579784" ixy="0.0" ixz="0.0" iyy="0.0047579784" iyz="0.0" izz="0.0047579784" />
+-->
+		<inertia ixx="0.3" ixy="0.0" ixz="0.0" iyy="0.3" iyz="0.0" izz="0.3" />
       </inertial>
       <!-- end for simulation -->
@@ -172,5 +187,8 @@
         <origin xyz="0 0 0" rpy="0 0 0" />
         <mass value="3.5" />
+<!--
         <inertia ixx="0.0068523756" ixy="0.0" ixz="0.0" iyy="0.0068523756" iyz="0.0" izz="0.0068523756" />
+-->
+		<inertia ixx="0.3" ixy="0.0" ixz="0.0" iyy="0.3" iyz="0.0" izz="0.3" />
       </inertial>
       <!-- end for simulation -->
@@ -202,5 +220,8 @@
         <origin xyz="0 0 0" rpy="0 0 0" />
         <mass value="1.47" />
+<!--
         <inertia ixx="0.0028760256" ixy="0.0" ixz="0.0" iyy="0.0028760256" iyz="0.0" izz="0.0028760256" />
+-->
+		<inertia ixx="0.3" ixy="0.0" ixz="0.0" iyy="0.3" iyz="0.0" izz="0.3" />
       </inertial>
       <!-- end for simulation -->
@@ -232,5 +253,8 @@
         <origin xyz="0 0 0" rpy="0 0 0" />
         <mass value="0.45" />
+<!--
         <inertia ixx="0.0008938776" ixy="0.0" ixz="0.0" iyy="0.0008938776" iyz="0.0" izz="0.0008938776" />
+-->
+		<inertia ixx="0.3" ixy="0.0" ixz="0.0" iyy="0.3" iyz="0.0" izz="0.3" />
       </inertial>
       <!-- end for simulation -->

Commit message: Adapt joint limits to real robots limitations

File: franka_description/robots/panda_arm.xacro (robot description, xacro)
@@ -68,5 +68,5 @@
       <child link="${arm_id}_link1"/>
       <axis xyz="0 0 1"/>
-      <limit effort="87" lower="-2.8973" upper="2.8973" velocity="2.1750"/>
+      <limit effort="87" lower="-2.8973" upper="2.8973" velocity="0.25"/> <!-- original vel limit: 2.1750 -->
       <!-- for simulation -->
       <dynamics damping="${joint_damping}"/>
@@ -101,5 +101,5 @@
       <child link="${arm_id}_link2"/>
       <axis xyz="0 0 1"/>
-      <limit effort="87" lower="-1.7628" upper="1.7628" velocity="2.1750"/>
+      <limit effort="87" lower="-1.7628" upper="1.7628" velocity="0.25"/> <!-- original vel limit: 2.1750 -->
       <!-- for simulation -->
       <dynamics damping="${joint_damping}"/>
@@ -134,5 +134,5 @@
       <child link="${arm_id}_link3"/>
       <axis xyz="0 0 1"/>
-      <limit effort="87" lower="-2.8973" upper="2.8973" velocity="2.1750"/>
+      <limit effort="87" lower="-2.8973" upper="2.8973" velocity="0.25"/> <!-- original vel limit: 2.1750 -->
       <!-- for simulation -->
       <dynamics damping="${joint_damping}"/>
@@ -167,5 +167,5 @@
       <child link="${arm_id}_link4"/>
       <axis xyz="0 0 1"/>
-      <limit effort="87" lower="-3.0718" upper="-0.0698" velocity="2.1750"/>
+      <limit effort="87" lower="-3.0718" upper="-0.0698" velocity="0.25"/> <!-- original vel limit: 2.1750 -->
       <!-- for simulation -->
       <dynamics damping="${joint_damping}"/>
@@ -200,5 +200,5 @@
       <child link="${arm_id}_link5"/>
       <axis xyz="0 0 1"/>
-      <limit effort="12" lower="-2.8973" upper="2.8973" velocity="2.6100"/>
+      <limit effort="12" lower="-2.8973" upper="2.8973" velocity="0.25"/> <!-- original vel limit: 2.6100 -->
       <!-- for simulation -->
       <dynamics damping="${joint_damping}"/>
@@ -233,5 +233,5 @@
       <child link="${arm_id}_link6"/>
       <axis xyz="0 0 1"/>
-      <limit effort="12" lower="-0.0175" upper="3.7525" velocity="2.6100"/>
+      <limit effort="12" lower="-0.0175" upper="3.7525" velocity="0.25"/> <!-- original vel limit: 2.6100 -->
       <!-- for simulation -->
       <dynamics damping="${joint_damping}"/>
@@ -266,5 +266,5 @@
       <child link="${arm_id}_link7"/>
       <axis xyz="0 0 1"/>
-      <limit effort="12" lower="-2.8973" upper="2.8973" velocity="2.6100"/>
+      <limit effort="12" lower="-2.8973" upper="2.8973" velocity="0.25"/> <!-- original vel limit: 2.6100 -->
       <!-- for simulation -->
       <dynamics damping="${joint_damping}"/>

Commit message: Reset joint velocities such that right in simulation; must be changed for real robot

File: franka_description/robots/panda_arm.xacro (robot description, xacro)
@@ -68,5 +68,5 @@
       <child link="${arm_id}_link1"/>
       <axis xyz="0 0 1"/>
-      <limit effort="87" lower="-2.8973" upper="2.8973" velocity="0.25"/> <!-- original vel limit: 2.1750 -->
+      <limit effort="87" lower="-2.8973" upper="2.8973" velocity="2.1750"/> <!-- reduce for real robot to 0.25  -->
       <!-- for simulation -->
       <dynamics damping="${joint_damping}"/>
@@ -101,5 +101,5 @@
       <child link="${arm_id}_link2"/>
       <axis xyz="0 0 1"/>
-      <limit effort="87" lower="-1.7628" upper="1.7628" velocity="0.25"/> <!-- original vel limit: 2.1750 -->
+      <limit effort="87" lower="-1.7628" upper="1.7628" velocity="2.1750"/> <!-- reduce for real robot to 0.25  -->
       <!-- for simulation -->
       <dynamics damping="${joint_damping}"/>
@@ -134,5 +134,5 @@
       <child link="${arm_id}_link3"/>
       <axis xyz="0 0 1"/>
-      <limit effort="87" lower="-2.8973" upper="2.8973" velocity="0.25"/> <!-- original vel limit: 2.1750 -->
+      <limit effort="87" lower="-2.8973" upper="2.8973" velocity="2.1750"/> <!-- reduce for real robot to 0.25  -->
       <!-- for simulation -->
       <dynamics damping="${joint_damping}"/>
@@ -167,5 +167,5 @@
       <child link="${arm_id}_link4"/>
       <axis xyz="0 0 1"/>
-      <limit effort="87" lower="-3.0718" upper="-0.0698" velocity="0.25"/> <!-- original vel limit: 2.1750 -->
+      <limit effort="87" lower="-3.0718" upper="-0.0698" velocity="2.1750"/> <!-- reduce for real robot to 0.25  -->
       <!-- for simulation -->
       <dynamics damping="${joint_damping}"/>
@@ -200,5 +200,5 @@
       <child link="${arm_id}_link5"/>
       <axis xyz="0 0 1"/>
-      <limit effort="12" lower="-2.8973" upper="2.8973" velocity="0.25"/> <!-- original vel limit: 2.6100 -->
+      <limit effort="12" lower="-2.8973" upper="2.8973" velocity="2.6100"/> <!-- reduce for real robot to 0.25  -->
       <!-- for simulation -->
       <dynamics damping="${joint_damping}"/>
@@ -233,5 +233,5 @@
       <child link="${arm_id}_link6"/>
       <axis xyz="0 0 1"/>
-      <limit effort="12" lower="-0.0175" upper="3.7525" velocity="0.25"/> <!-- original vel limit: 2.6100 -->
+      <limit effort="12" lower="-0.0175" upper="3.7525" velocity="2.6100"/> <!-- reduce for real robot to 0.25  -->
       <!-- for simulation -->
       <dynamics damping="${joint_damping}"/>
@@ -266,5 +266,5 @@
       <child link="${arm_id}_link7"/>
       <axis xyz="0 0 1"/>
-      <limit effort="12" lower="-2.8973" upper="2.8973" velocity="0.25"/> <!-- original vel limit: 2.6100 -->
+      <limit effort="12" lower="-2.8973" upper="2.8973" velocity="2.6100"/> <!-- reduce for real robot to 0.25  -->
       <!-- for simulation -->
       <dynamics damping="${joint_damping}"/>
